File: relay16.kicad_pcb (KiCad board)
At the start: 2 copper layers, 154 x 93 mm, 119 parts, among them J1 Screw_Terminal_01x03, J10 Screw_Terminal_01x03, J11 Screw_Terminal_01x03, J12 Screw_Terminal_01x03, J13 Screw_Terminal_01x03, J14 Screw_Terminal_01x03, J15 Screw_Terminal_01x03, J16 Screw_Terminal_01x03, J17 Screw_Terminal_01x02, J2 Screw_Terminal_01x03, J3 Screw_Terminal_01x03, J4 Screw_Terminal_01x03, J5 Screw_Terminal_01x03, J6 Screw_Terminal_01x03, J7 Screw_Terminal_01x03, J8 Screw_Terminal_01x03, J9 Screw_Terminal_01x03, K1 SANYOU_SRD_Form_C, K10 SANYOU_SRD_Form_C, K11 SANYOU_SRD_Form_C, K12 SANYOU_SRD_Form_C, K13 SANYOU_SRD_Form_C, K14 SANYOU_SRD_Form_C, K15 SANYOU_SRD_Form_C, K16 SANYOU_SRD_Form_C, K2 SANYOU_SRD_Form_C, K3 SANYOU_SRD_Form_C, K4 SANYOU_SRD_Form_C, K5 SANYOU_SRD_Form_C, K6 SANYOU_SRD_Form_C, K7 SANYOU_SRD_Form_C, K8 SANYOU_SRD_Form_C, K9 SANYOU_SRD_Form_C, Q1 2N7002E, Q10 2N7002E, Q11 2N7002E, Q12 2N7002E, Q13 2N7002E, Q14 2N7002E, Q15 2N7002E, Q16 2N7002E, Q2 2N7002E, Q3 2N7002E, Q4 2N7002E, Q5 2N7002E, Q6 2N7002E, Q7 2N7002E, Q8 2N7002E, Q9 2N7002E

Commit message: Data as ordered.
Parts:
- added TP1: TestPoint, TestPoint:TestPoint_Pad_2.5x2.5mm, B.Cu at (96.5, 59.8)
- added TP10: TestPoint, TestPoint:TestPoint_Pad_2.5x2.5mm, B.Cu at (191.5, 128.5)
- added TP11: TestPoint, TestPoint:TestPoint_Pad_2.5x2.5mm, B.Cu at (174.0, 128.5)
- added TP12: TestPoint, TestPoint:TestPoint_Pad_2.5x2.5mm, B.Cu at (156.5, 128.5)
- added TP13: TestPoint, TestPoint:TestPoint_Pad_2.5x2.5mm, B.Cu at (86.5, 55.8)
- added TP14: TestPoint, TestPoint:TestPoint_Pad_2.5x2.5mm, B.Cu at (104.0, 55.8)
- added TP15: TestPoint, TestPoint:TestPoint_Pad_2.5x2.5mm, B.Cu at (121.5, 55.8)
- added TP16: TestPoint, TestPoint:TestPoint_Pad_2.5x2.5mm, B.Cu at (139.0, 55.8)
- added TP17: TestPoint, TestPoint:TestPoint_Pad_2.5x2.5mm, B.Cu at (156.5, 55.8)
- added TP18: TestPoint, TestPoint:TestPoint_Pad_2.5x2.5mm, B.Cu at (174.0, 55.8)
- added TP19: TestPoint, TestPoint:TestPoint_Pad_2.5x2.5mm, B.Cu at (191.5, 55.8)
- added TP2: TestPoint, TestPoint:TestPoint_Pad_2.5x2.5mm, B.Cu at (114.0, 59.8)
- added TP20: TestPoint, TestPoint:TestPoint_Pad_2.5x2.5mm, B.Cu at (209.0, 55.8)
- added TP21: TestPoint, TestPoint:TestPoint_Pad_2.5x2.5mm, B.Cu at (219.0, 132.2)
- added TP22: TestPoint, TestPoint:TestPoint_Pad_2.5x2.5mm, B.Cu at (201.5, 132.2)
- added TP23: TestPoint, TestPoint:TestPoint_Pad_2.5x2.5mm, B.Cu at (184.0, 132.2)
- added TP24: TestPoint, TestPoint:TestPoint_Pad_2.5x2.5mm, B.Cu at (166.5, 132.2)
- added TP25: TestPoint, TestPoint:TestPoint_Pad_2.5x2.5mm, B.Cu at (139.0, 128.5)
- added TP26: TestPoint, TestPoint:TestPoint_Pad_2.5x2.5mm, B.Cu at (121.5, 128.5)
- added TP27: TestPoint, TestPoint:TestPoint_Pad_2.5x2.5mm, B.Cu at (104.0, 128.2)
- added TP28: TestPoint, TestPoint:TestPoint_Pad_2.5x2.5mm, B.Cu at (86.5, 128.2)
- added TP29: TestPoint, TestPoint:TestPoint_Pad_2.5x2.5mm, B.Cu at (149.2, 132.2)
- added TP3: TestPoint, TestPoint:TestPoint_Pad_2.5x2.5mm, B.Cu at (131.5, 59.8)
- added TP30: TestPoint, TestPoint:TestPoint_Pad_2.5x2.5mm, B.Cu at (131.5, 132.2)
- added TP31: TestPoint, TestPoint:TestPoint_Pad_2.5x2.5mm, B.Cu at (114.0, 132.2)
- added TP32: TestPoint, TestPoint:TestPoint_Pad_2.5x2.5mm, B.Cu at (96.5, 132.2)
- added TP4: TestPoint, TestPoint:TestPoint_Pad_2.5x2.5mm, B.Cu at (149.0, 59.8)
- added TP5: TestPoint, TestPoint:TestPoint_Pad_2.5x2.5mm, B.Cu at (166.5, 59.8)
- added TP6: TestPoint, TestPoint:TestPoint_Pad_2.5x2.5mm, B.Cu at (184.0, 59.8)
- added TP7: TestPoint, TestPoint:TestPoint_Pad_2.5x2.5mm, B.Cu at (201.5, 59.8)
- added TP8: TestPoint, TestPoint:TestPoint_Pad_2.5x2.5mm, B.Cu at (219.0, 59.8)
- added TP9: TestPoint, TestPoint:TestPoint_Pad_2.5x2.5mm, B.Cu at (209.0, 128.5)
Other:
- board text added: "Serial: 115200 SERIAL_8N1$ Comamnd: 16bit hex string from {dblquote}0000{dblquote} to {dblquote}FFFF{dblquote} Termination: {dblquote}\r{dblquote} or {dblquote}\r\n{dblquote}"
- board text removed: "Serial: 115200 SERIAL_8N1 CH_X ON: {dblquote}X+\r\n{dblquote} CH_X OFF: {dblquote}X-\r\n{dblquote} All OFF: {dblquote}0-1-2-3-4-5-6-7-8-9-A-B-C-D-E-F-\r\n{dblquote} All ON: {dblquote}0-1+2+3+4+5+6+7+8+9+A+B+C+D+E+F+\r\n{dblquote} Response: Echo chars if ok, {dblquote}\r\n{dblquote} otherwise."
